Commit message: Control

File: rhobetto/robot.urdf (robot description, URDF)
Before this commit: robot rhobetto, 19 links, 18 joints
Links:
- added link left, mass 1e-9
- added link left_ankle_1, mass 1e-9
- added link left_ankle_2, mass 1e-9
- added link left_knee_1, mass 1e-9
- added link left_knee_2, mass 1e-9
- added link right, mass 1e-9
- added link right_ankle_1, mass 1e-9
- added link right_ankle_2, mass 1e-9
- added link right_knee_1, mass 1e-9
- added link right_knee_2, mass 1e-9
- added link trunk, mass 1e-9
- link dbl_pulley__list_yllcdchy6onwiy_default: mass 0.20962385689835016933 -> 0.20962385689835014158
- link dbl_pulley__list_yllcdchy6onwiy_default_4: mass 0.20962385689835016933 -> 0.20962385689835014158
- link hip: mass 0.99833109183451718138 -> 0.9983310918345172924
- link hip_2: mass 0.99833109183451740343 -> 0.99833109183451762547
- link left_tibia: mass 0.37331562544444790719 -> 0.3733156254444479627
- link motor_pulley__list_kldlfi9cxi833p__80_4: mass 0.41210159105458799012 -> 0.41210159105458804563
- link pelvis: mass 1.8817862296976988201 -> 1.881786229697698376
- link right_foot: mass 0.21580776100670012729 -> 0.21580776100670015505
Joints:
- added joint left_ankle_1_frame: type fixed, parent dbl_pulley__list_yllcdchy6onwiy_default_2, child left_ankle_1, origin xyz=1.249000902703301108e-16 5.5511151231257827021e-17 -0.045000000000000178746 rpy=-1.5707963267948898967 8.2106794746731389155e-17 -2.626030194172424892, axis 0 0 0
- added joint left_ankle_2_frame: type fixed, parent left_foot, child left_ankle_2, origin xyz=1.2767564783189300215e-15 1.0963452368173420837e-15 -0.012999999999992045696 rpy=-1.5707963267949809349 8.1712414612412783553e-14 1.5707963267948445996, axis 0 0 0
- added joint left_frame: type fixed, parent left_foot, child left, origin xyz=0.037000000000000476952 0.030092322087891358595 0.0092500000000063642425 rpy=-1.5707963267949796027 8.1601392309949687297e-14 1.5707963267948361619, axis 0 0 0
- added joint left_knee_1_frame: type fixed, parent dbl_pulley__list_yllcdchy6onwiy_default, child left_knee_1, origin xyz=-2.3592239273284576484e-16 -1.9428902930940239457e-16 -0.044999999999995030087 rpy=-1.570796326794896336 -1.9312549720731026129e-16 -2.626030194172424892, axis 0 0 0
- added joint left_knee_2_frame: type fixed, parent left_tibia, child left_knee_2, origin xyz=4.4408920985006261617e-16 -2.2690183065776636795e-15 -0.027500000000002675082 rpy=-1.5707963267948770181 -6.826483822663960308e-14 -1.5707963267947628871, axis 0 0 0
- added joint right_ankle_1_frame: type fixed, parent dbl_pulley__list_yllcdchy6onwiy_default_4, child right_ankle_1, origin xyz=5.5511151231257827021e-17 0 -0.045000000000000039968 rpy=1.5707963267948974462 -4.4381033991324517763e-17 -1.1999662206236612061, axis 0 0 0
- added joint right_ankle_2_frame: type fixed, parent right_foot, child right_ankle_2, origin xyz=-1.1102230246251565404e-16 -4.1633363423443370266e-17 -0.012999999999999720113 rpy=1.570796326794896558 -7.6289165872435842086e-31 -1.570796326794896558, axis 0 0 0
- added joint right_frame: type fixed, parent right_foot, child right, origin xyz=0.036999999999999977351 -0.030092322087891410637 0.0092500000000002996492 rpy=1.57079632679489678 -6.2623444500028930906e-31 -1.570796326794896336, axis 0 0 0
- added joint right_knee_1_frame: type fixed, parent dbl_pulley__list_yllcdchy6onwiy_default_3, child right_knee_1, origin xyz=-1.8041124150158793782e-16 5.5511151231257827021e-17 -0.045000000000001233458 rpy=1.570796326794896558 1.5521297560595994805e-16 0.37083010617123557395, axis 0 0 0
- added joint right_knee_2_frame: type fixed, parent right_tibia, child right_knee_2, origin xyz=0 2.0816681711721685133e-17 -0.02750000000000005218 rpy=1.5707963267948921171 -7.2164496600631990102e-16 1.5707963267948898967, axis 0 0 0
- added joint trunk_frame: type fixed, parent pelvis, child trunk, origin xyz=3.1918911957973250537e-16 0.039500096321092123541 0.2763194116985674964 rpy=-4.9303806576313237838e-32 1.2246467991473529607e-16 -1.570796326794896558, axis 0 0 0
- joint left_ankle_1: origin xyz=0 0.10000000000000006106 0.031699914169307799594 rpy=3.1415926535897922278 1.1796119636658898694e-16 3.1415926535897917837 -> xyz=-1.43288159115684266e-14 0.10000000000003941847 0.031699914169318055279 rpy=-3.1415926535896332439 2.7698801309900253552e-13 -2.6260301991139058941
- joint left_ankle_2: origin xyz=2.7755575615628913511e-17 0.23000000000000003775 0.017200010490399944563 rpy=3.1415926535897917837 1.7324509531491014183e-28 3.1415926535897917837 -> xyz=2.7755575615628913511e-17 0.23000000000000000999 0.01720001049039995844 rpy=-3.1415926535897837901 -5.0396915472993869245e-15 -2.6260301991139489708
- joint left_ankle_3: origin xyz=-0.19800000000000034239 3.2612801348363973375e-16 0.014500000000000012879 rpy=-1.9322831681911389219e-14 -1.1952702991551301084e-14 3.1415926535897917837 -> xyz=-0.19800000000000050893 -2.5902890943285683534e-14 0.01449999999999404543 rpy=5.5164206536062055395e-14 2.071137857571814068e-14 -3.1415926535897713556
- joint left_hip_pitch: origin xyz=0.039499999999980127396 -1.8457457784393227485e-15 -0.074699998778100198948 rpy=3.141592653589793116 1.5707963267948930053 0 -> xyz=0.039499999999983950727 -1.7486012637846215512e-15 -0.074699998778100115682 rpy=3.1415926535897926719 1.5707963267948947816 0
- joint left_hip_roll_2: origin xyz=0.094654092773412482065 0.11429998950959337212 -0.035999999999999719724 rpy=1.5707963267948976682 1.7634439393673709815e-14 -3.1415926535897922278 -> xyz=0.094654092773413786577 0.11429998950959213699 -0.035999999999999539313 rpy=1.5707963267948978903 -0 -3.1415926535897913396
- joint left_knee_1: origin xyz=-0.039499999999977442044 8.9511731360403246072e-16 -0.074699998778100046293 rpy=-3.141592653589793116 -1.5707963267948927832 0 -> xyz=-0.039499999999981591503 1.103284130721249312e-15 -0.074699998778099963026 rpy=3.1415926535897926719 -1.5707963267948945596 0
- joint left_knee_2: origin xyz=0 0.13400000000000000799 0.066199903678899926773 rpy=3.1415926535897877869 2.9837243786650480588e-15 -3.141592653589793116 -> xyz=0 0.13399999999999998024 0.066199903678899912896 rpy=-3.141592653589788231 -2.076894388873911815e-15 -2.6260301991139525235
- joint left_knee_3: origin xyz=2.7755575615628913511e-17 0.22999999999999998224 0.066199903678899912896 rpy=-3.1415926535897904515 -1.7158652907544210928e-30 -1.570796326794896558 -> xyz=2.7755575615628913511e-17 0.23000000000000000999 0.066199903678899968407 rpy=3.1415926535897917837 -4.3853809472694693089e-15 -1.570796326794896558
- joint right_ankle_1: origin xyz=6.9388939039072283776e-18 -0.10000000000000000555 0.031699914169307799594 rpy=-3.1415926535897873428 -8.725778676316278914e-15 -2.7707548731624784821 -> xyz=-6.9388939039072283776e-18 -0.10000000000000000555 0.0316999141693077649 rpy=-3.1415926535897873428 -8.725778676316278914e-15 -2.7707548731624784821
- joint right_ankle_2: origin xyz=-2.0816681711721685133e-17 -0.2300000000000000655 0.017200010490399916807 rpy=3.1415926535897886751 -8.1964432562112751426e-15 -1.199958546367576373 -> xyz=2.7755575615628913511e-17 -0.2300000000000000655 0.017200010490399923746 rpy=3.1415926535897886751 -8.196443256211278298e-15 -1.199958546367576373
- joint right_ankle_3: origin xyz=-0.19800000000001038991 -1.3877787807814456755e-17 0.014499999999999277356 rpy=7.288047944146430554e-15 1.8368469868820638049e-14 3.1415926535897837901 -> xyz=-0.19800000000000267386 -1.3877787807814456755e-17 0.014500000000001012079 rpy=-1.929779299638754658e-15 3.8030946983891268802e-16 3.1415926535897837901
- joint right_hip_pitch: origin xyz=0.039499999999982007837 -7.147060721024445229e-16 -0.07469999877810150346 rpy=1.1948705341884184515e-16 -1.5707963267948936714 0 -> xyz=0.039499999999982007837 -7.8409501114151680667e-16 -0.074699998778101545094 rpy=2.8327694488241544824e-16 -1.5707963267948938935 0
- joint right_knee_2: origin xyz=-4.8572257327350598644e-17 -0.13400000000000000799 0.066199903678899843507 rpy=3.1415926535897851224 4.4358406448577547666e-15 0.37083778042732185032 -> xyz=0 -0.13400000000000003575 0.066199903678899857384 rpy=3.1415926535897851224 4.4436446934595034556e-15 0.37083778042730392022
- joint right_knee_3: origin xyz=2.7755575615628913511e-17 -0.23000000000000000999 0.066199903678899899018 rpy=-3.1415926535897873428 2.6181831849055039216e-30 1.570796326794896558 -> xyz=3.4694469519536141888e-17 -0.22999999999999995448 0.06619990367889988514 rpy=-3.1415926535897877869 8.8193055618606019435e-15 1.570796326794896558
