Commit message: Rhobetto V2

File: rhobetto/robot.urdf (robot description, URDF)
Before this commit: robot rhobetto, 30 links, 29 joints
Links:
- removed link dbl_pulley__list_yllcdchy6onwiy_default
- removed link dbl_pulley__list_yllcdchy6onwiy_default_2
- removed link dbl_pulley__list_yllcdchy6onwiy_default_3
- removed link dbl_pulley__list_yllcdchy6onwiy_default_4
- removed link hip
- removed link hip_2
- removed link left_ankle_1
- removed link left_ankle_2
- removed link left_knee_1
- removed link left_knee_2
- removed link motor_pulley__list_kldlfi9cxi833p__80
- removed link motor_pulley__list_kldlfi9cxi833p__80_2
- removed link motor_pulley__list_kldlfi9cxi833p__80_3
- removed link motor_pulley__list_kldlfi9cxi833p__80_4
- removed link motor_pulley__list_kldlfi9cxi833p__80_5
- removed link motor_pulley__list_kldlfi9cxi833p__80_6
- removed link right_ankle_1
- removed link right_ankle_2
- removed link right_knee_1
- removed link right_knee_2
- added link ankle_shaft, mass 0.027812191526678471665; collision mesh filename=package:///ankle_shaft.stl; collision mesh filename=package:///shaft_end.stl
- added link ankle_shaft_2, mass 0.027812191526678475134; collision mesh filename=package:///ankle_shaft.stl; collision mesh filename=package:///shaft_end.stl
- added link closing_left_1, mass 1e-9
- added link closing_left_2, mass 1e-9
- added link closing_right_1, mass 1e-9
- added link closing_right_2, mass 1e-9
- added link left_ankle, mass 0.03015568460546654006; collision mesh filename=package:///ankle_alu.stl; collision mesh filename=package:///ankle_alu.stl
- added link left_lower_hip, mass 0.37002551285788642943; collision mesh filename=package:///inner_hip.stl; collision mesh filename=package:///rmd_x6.stl
- added link left_shaft_connector, mass 0.061135779919446485431; collision mesh filename=package:///asc_2_mirror.stl; collision mesh filename=package:///asc_alu.stl
- added link left_upper_hip, mass 0.47353711718592900182; collision mesh filename=package:///bearing_cover_1.stl; collision mesh filename=package:///bearing_cover_1.stl
- added link motor_pulley, mass 0.068767168773007744664; collision mesh filename=package:///motor_pulley.stl; visual mesh filename=package:///motor_pulley.stl
- added link motor_pulley_2, mass 0.068767168773007744664; collision mesh filename=package:///motor_pulley.stl; visual mesh filename=package:///motor_pulley.stl
- added link motor_pulley_3, mass 0.068767168773007730787; collision mesh filename=package:///motor_pulley.stl; visual mesh filename=package:///motor_pulley.stl
- added link motor_pulley_4, mass 0.068767168773007744664; collision mesh filename=package:///motor_pulley.stl; visual mesh filename=package:///motor_pulley.stl
- added link motor_pulley_5, mass 0.068767168773007744664; collision mesh filename=package:///motor_pulley.stl; visual mesh filename=package:///motor_pulley.stl
- added link motor_pulley_6, mass 0.068767168773007730787; collision mesh filename=package:///motor_pulley.stl; visual mesh filename=package:///motor_pulley.stl
- added link right_ankle, mass 0.030363454605670948949; collision mesh filename=package:///ankle.stl; collision mesh filename=package:///ankle_alu.stl
- added link right_lower_hip, mass 0.38603836162425869682; collision mesh filename=package:///inner_hip_mirror.stl; collision mesh filename=package:///rmd_x6.stl
- added link right_shaft_connector, mass 0.061462040916151317038; collision mesh filename=package:///asc_2.stl; collision mesh filename=package:///asc_alu.stl
- added link right_upper_hip, mass 0.47353718531678168358; collision mesh filename=package:///bearing_cover_1.stl; collision mesh filename=package:///bearing_cover_1.stl
- link left_femur: mass 0.7913553249145355295 -> 0.86687774720833488118; geometry collision mesh filename=package:///bearing_cover_1.stl; collision mesh filename=package:///bearing_cover_2.stl
- link left_foot: mass 0.2163573891864303822 -> 0.055361091085330056683; geometry collision mesh filename=package:///foot_alu.stl; collision mesh filename=package:///lower_foot_mirror.stl
- link left_tibia: mass 0.3733156254444479627 -> 0.13716146838378595607; geometry collision mesh filename=package:///inner_tibia.stl; collision mesh filename=package:///outer_knee_1.stl
- link pelvis: mass 1.881786229697698376 -> 0.51681395261861506896; geometry collision mesh filename=package:///pelvis.stl; collision mesh filename=package:///pelvis_bearing_housing.stl
- link right_femur: mass 0.79097151548500232998 -> 0.86662877599053789179; geometry collision mesh filename=package:///bearing_cover_1.stl; collision mesh filename=package:///bearing_cover_2.stl
- link right_foot: mass 0.21580776100670015505 -> 0.055361091085330049744; geometry collision mesh filename=package:///foot_alu.stl; collision mesh filename=package:///lower_foot.stl
- link right_tibia: mass 0.37356459666752256377 -> 0.13703698277488743362; geometry collision mesh filename=package:///inner_tibia.stl; collision mesh filename=package:///outer_knee_1_mirror.stl
Joints:
- removed joint left_ankle_1
- removed joint left_ankle_1_frame
- removed joint left_ankle_2
- removed joint left_ankle_2_frame
- removed joint left_ankle_3
- removed joint left_knee_1_frame
- removed joint left_knee_2_frame
- removed joint left_knee_3
- removed joint right_ankle_1
- removed joint right_ankle_1_frame
- removed joint right_ankle_2
- removed joint right_ankle_2_frame
- removed joint right_ankle_3
- removed joint right_knee_1_frame
- removed joint right_knee_2_frame
- removed joint right_knee_3
- added joint closing_left_1_frame: type fixed, parent ankle_shaft, child closing_left_1, origin xyz=-0.14999999999999771849 -0.050000000000000030531 -6.4531713306337223912e-16 rpy=-9.9920072216398766916e-16 -1.8870233948204239244e-15 -6.3481963726237970789e-15, axis 0 0 0
- added joint closing_left_2_frame: type fixed, parent left_ankle, child closing_left_2, origin xyz=0.024999999999998648303 4.9960036108132044319e-16 -0.023800000000004244843 rpy=-7.5065461826747186547e-16 1.3561226421362389337e-16 -3.1415926535897926719, axis 0 0 0
- added joint closing_right_1_frame: type fixed, parent right_ankle, child closing_right_1, origin xyz=0.024999999999999994449 -1.1102230246251565404e-16 -0.020999903678907916316 rpy=-7.3769885253638019017e-17 -2.4589961751229850247e-17 2.3112295755706704928e-29, axis 0 0 0
- added joint closing_right_2_frame: type fixed, parent ankle_shaft_2, child closing_right_2, origin xyz=-0.14999999999999633071 -0.049999999999998864797 -0.0069999999999999784617 rpy=1.3103514549253502123e-28 -9.3797041067719513922e-16 3.1415926535897895633, axis 0 0 0
- added joint left_ankle_pitch_1: type revolute, parent left_femur, child motor_pulley_3, origin xyz=3.3323121855078318776e-15 -0.080000000000102614028 0.018300000000037931758 rpy=1.215759610759047731e-14 -1.1177312336507953765e-13 3.0929397216733969245, axis 0 0 1, limit effort=1 velocity=20
- added joint left_ankle_pitch_2: type revolute, parent left_tibia, child left_shaft_connector, origin xyz=3.5319520210675786405e-15 2.5812685322534889565e-14 -0.048799903678906839111 rpy=3.1415926535896776528 -1.2602542893967900286e-13 -1.5707963268030824544, axis 0 0 1, limit lower=-1.2375158973761830605 upper=1.570796326794896558 effort=1 velocity=20
- added joint left_ankle_pitch_3: type revolute, parent left_shaft_connector, child ankle_shaft, origin xyz=-8.8817841970012523234e-16 -0.025000000000006249862 -0.023800000000064245459 rpy=-1.0941417982723899411e-14 -2.9892138505736365462e-14 3.1415926535816263154, axis 0 0 1, limit effort=1 velocity=20
- added joint left_ankle_pitch_4: type revolute, parent left_tibia, child left_ankle, origin xyz=7.4904621468630412097e-15 -0.15000000000016919244 -0.048799903678869403778 rpy=-3.1415926535896323557 -1.077999630545015724e-13 -3.1415926535897318317, axis 0 0 1, limit lower=-1.2375158973761830605 upper=1.570796326794896558 effort=1 velocity=20
- added joint left_ankle_roll: type revolute, parent left_ankle, child left_foot, origin xyz=-0.0065000000000031482247 -0.032500000000081408214 -0.027299999999997218852 rpy=6.804680578063719959e-27 1.570796326794891673 0, axis 0 0 1, limit lower=-0.1745329251994329478 upper=0.52359877559829881566 effort=1 velocity=20
- added joint left_hip_yaw: type revolute, parent pelvis, child left_upper_hip, origin xyz=0.0093499908672946222682 -0.061399903678804698681 0.17949999877806774307 rpy=3.1415926535895537519 4.2659356562086370119e-16 3.7448197579691025492e-14, axis 0 0 1, limit lower=-1.570796326794896558 upper=1.570796326794896558 effort=1 velocity=20
- added joint right_ankle_pitch_1: type revolute, parent right_femur, child motor_pulley_6, origin xyz=-4.8647140664784363295e-13 0.080000000000202506345 0.018299999999978916465 rpy=4.4539911443551959561e-16 -1.9360994195986860955e-15 -1.1372251246499935906, axis 0 0 1, limit effort=1 velocity=20
- added joint right_ankle_pitch_2: type revolute, parent right_tibia, child right_shaft_connector, origin xyz=1.3883013479743998971e-14 9.7893915196323177952e-14 -0.048799903678874739787 rpy=3.1415926535897300553 6.9485480086530627972e-14 1.5707963267882383285, axis 0 0 1, limit lower=-1.570796326794896558 upper=1.2375158973761830605 effort=1 velocity=20
- added joint right_ankle_pitch_3: type revolute, parent right_shaft_connector, child ankle_shaft_2, origin xyz=5.7537308251198737707e-14 0.02499999999997508035 -0.030799903678917495142 rpy=-3.1415926535897793492 7.2586854802179579745e-15 3.1415926535832938704, axis 0 0 1, limit effort=1 velocity=20
- added joint right_ankle_pitch_4: type revolute, parent right_tibia, child right_ankle, origin xyz=4.6832013725719971683e-16 0.15000000000000299205 -0.0040000000000158519864 rpy=6.9436156178235627099e-14 6.3059604428588073261e-14 -3.141592653589638573, axis 0 0 1, limit lower=-1.2375158973761830605 upper=1.570796326794896558 effort=1 velocity=20
- added joint right_ankle_roll: type revolute, parent right_ankle, child right_foot, origin xyz=-0.0065000000000001272038 -0.032499999999999029665 -0.01749990367890758014 rpy=-1.6386994296483263268e-27 1.5707963267948956698 0, axis 0 0 1, limit lower=-0.52359877559829881566 upper=0.1745329251994329478 effort=1 velocity=20
- added joint right_hip_yaw: type revolute, parent pelvis, child right_upper_hip, origin xyz=0.0093499908672991186714 -0.18139990367880462485 0.1794999987780965256 rpy=-3.1415926535895533078 -4.5025549804522808348e-16 3.1415926535897784611, axis 0 0 1, limit lower=-1.570796326794896558 upper=1.570796326794896558 effort=1 velocity=20
- joint left_frame: origin xyz=0.037000000000000476952 0.030092322087891358595 0.0092500000000063642425 rpy=-1.5707963267949796027 8.1601392309949687297e-14 1.5707963267948361619 -> xyz=2.7956803538842223134e-14 -0.018500000000039928949 -0.00075698915672654798481 rpy=-1.5707963267948510389 1.5707963267948410468 0
- joint left_hip_pitch: limit lower=-0.61086523819801530344 upper=0.61086523819801530344 effort=1 velocity=20 -> lower=-1.0471975511965976313 upper=1.9198621771937625091 effort=1 velocity=20; origin xyz=0.039499999999983950727 -1.7486012637846215512e-15 -0.074699998778100115682 rpy=3.1415926535897926719 1.5707963267948947816 0 -> xyz=0.028499903678899887738 0.057999998778099942642 -0.026999998778100064295 rpy=3.141592653589793116 1.5707963267948190644 0; parent hip -> left_lower_hip
- joint left_hip_roll_1: child motor_pulley__list_kldlfi9cxi833p__80 -> motor_pulley; origin xyz=-2.9247893113481567484e-16 -4.8572257327350598644e-17 5.5855902341423913134e-16 rpy=-1.5707963267948978903 9.8051515370203805957e-32 1.8653968723158184032e-15 -> xyz=-0.011249993324299658107 -3.3334446314370325126e-14 0.066500000000009912293 rpy=-1.5707963267948970021 -2.6313752692175340574e-17 -1.5707963267953473085; parent pelvis -> left_upper_hip
- joint left_hip_roll_2: child hip -> left_lower_hip; limit lower=-0.785398163397448279 upper=0.43633231299858238339 effort=1 velocity=20 -> lower=-1.0471975511965976313 upper=0.1745329251994329478 effort=1 velocity=20; origin xyz=0.094654092773413786577 0.11429998950959213699 -0.035999999999999539313 rpy=1.5707963267948978903 -0 -3.1415926535897913396 -> xyz=-0.036349989645404076621 -2.9155150516047001474e-13 0.12149999999995617084 rpy=1.5707963267948956698 -1.871157079710716612e-14 -1.570796326794792197; parent pelvis -> left_upper_hip
- joint left_knee_1: child motor_pulley__list_kldlfi9cxi833p__80_3 -> motor_pulley_2; origin xyz=-0.039499999999981591503 1.103284130721249312e-15 -0.074699998778099963026 rpy=3.1415926535897926719 -1.5707963267948945596 0 -> xyz=-6.4989503856405845926e-16 -4.7361719415863419403e-15 -0.032900000000045240278 rpy=-3.1415926535897735761 -2.1496217883359487372e-16 0.027203981649072464521; parent hip -> left_femur
- joint left_knee_2: child dbl_pulley__list_yllcdchy6onwiy_default -> left_tibia; limit effort=1 velocity=20 -> lower=-2.356194490192344837 upper=0 effort=1 velocity=20; origin xyz=0 0.13399999999999998024 0.066199903678899912896 rpy=-3.141592653589788231 -2.076894388873911815e-15 -2.6260301991139525235 -> xyz=9.2534826152769928882e-15 -0.15000000000019156343 0.046499903679005291646 rpy=2.7514247754725331809e-15 8.3266726844769289951e-16 -2.997079401201851963e-16
- joint right_frame: origin xyz=0.036999999999999977351 -0.030092322087891410637 0.0092500000000002996492 rpy=1.57079632679489678 -6.2623444500028930906e-31 -1.570796326794896336 -> xyz=8.3266726846886740532e-17 -0.018500000000000182965 -0.00075698915673005212623 rpy=-1.570796326794896558 1.570796326794896558 0
- joint right_hip_pitch: limit lower=-0.61086523819801530344 upper=0.61086523819801530344 effort=1 velocity=20 -> lower=-1.9198621771937625091 upper=1.0471975511965976313 effort=1 velocity=20; origin xyz=0.039499999999982007837 -7.8409501114151680667e-16 -0.074699998778101545094 rpy=2.8327694488241544824e-16 -1.5707963267948938935 0 -> xyz=-0.028499903678899846104 0.057999998778099991215 -0.026999998778099998376 rpy=6.1232339957388072135e-17 1.570796326794896558 0; parent hip_2 -> right_lower_hip
- joint right_hip_roll_1: child motor_pulley__list_kldlfi9cxi833p__80_4 -> motor_pulley_4; origin xyz=-4.5267768468486773323e-16 0.078999999999999931388 4.5523838501157857761e-16 rpy=-1.5707963267948952257 -7.0516107484398242171e-30 -3.1415926535897913396 -> xyz=0.011249993324321095819 4.7184478546569152968e-15 0.066499999999996894928 rpy=1.5707963267948947816 -1.1323782996484244023 -1.5707963267948938935; parent pelvis -> right_upper_hip
- joint right_hip_roll_2: child hip_2 -> right_lower_hip; limit lower=-0.785398163397448279 upper=0.43633231299858238339 effort=1 velocity=20 -> lower=-0.1745329251994329478 upper=1.0471975511965976313 effort=1 velocity=20; origin xyz=-0.094654092773414452711 -0.035299989509592018255 -0.035999999999999358902 rpy=1.5707963267948952257 -9.5892432233253569701e-15 1.8653968745086079617e-15 -> xyz=0.036349989645413194328 2.9420910152566648321e-15 0.12149999999999683276 rpy=1.5707963267948972241 -1.3553674556756956347e-13 1.5707963267948970021; parent pelvis -> right_upper_hip
- joint right_knee_1: child motor_pulley__list_kldlfi9cxi833p__80_6 -> motor_pulley_5; origin xyz=-0.03949999999998299316 4.5796699765787707292e-16 -0.074699998778101517338 rpy=3.141592653589793116 -1.570796326794886788 0 -> xyz=-1.3617031301289482367e-16 -2.0852227908145500428e-15 -0.03289999999999071445 rpy=-3.141592653589793116 1.7432697531983926309e-15 2.0043675289397979711; parent hip_2 -> right_femur
- joint right_knee_2: child dbl_pulley__list_yllcdchy6onwiy_default_3 -> right_tibia; limit effort=1 velocity=20 -> lower=0 upper=2.356194490192344837 effort=1 velocity=20; origin xyz=0 -0.13400000000000003575 0.066199903678899857384 rpy=3.1415926535897851224 4.4436446934595034556e-15 0.37083778042730392022 -> xyz=-4.922167006389468494e-13 0.15000000000018082202 0.046499903678870690982 rpy=-8.733564085496093242e-16 2.1743913325908184736e-16 7.2423944486828269001e-13
- joint trunk_frame: origin xyz=3.1918911957973250537e-16 0.039500096321092123541 0.2763194116985674964 rpy=-4.9303806576313237838e-32 1.2246467991473529607e-16 -1.570796326794896558 -> xyz=0.0093499908672967854684 -0.12145115613833781798 0.17549999877808217241 rpy=-2.3968608495115065641e-13 1.224646799220653916e-16 3.7448197579713195639e-14
